Commit message: Updated

File: openDog_full.urdf (robot description, URDF)
Before this commit: robot opendog, 28 links, 26 joints
Joints:
- joint M10TibiaLinkage1.1: origin xyz=0 0. 0 rpy=0 0 0  -> xyz=0 0 0 rpy=0 0 0 
- joint M10TibiaLinkage1.2: origin xyz=0 0. 0 rpy=0 0 0  -> xyz=0 0 0 rpy=0 0 0 

Commit message: Update openDog_full.urdf

File: openDog_full.urdf (robot description, URDF)
Before this commit: robot opendog, 15 links, 14 joints
Links:
- added link M10LinkageFemur1.1_1, mass 0.1; collision cylinder length=0.21 radius=0.005; visual cylinder length=0.105 radius=0.005
- added link M10LinkageFemur1.1_2, mass 0.1; collision cylinder length=0.21 radius=0.005; visual cylinder length=0.105 radius=0.005
- added link M10ScrewFemur1.1, mass 0; collision cylinder length=0.05 radius=0.005; visual cylinder length=0.05 radius=0.005
- added link M10ScrewFemur1.2, mass 0; collision cylinder length=0.05 radius=0.005; visual cylinder length=0.05 radius=0.005
- added link M10ScrewFemur1.3, mass 0; collision cylinder length=0.05 radius=0.005; visual cylinder length=0.05 radius=0.005
- added link M10ScrewFemur1.4, mass 0; collision cylinder length=0.05 radius=0.005; visual cylinder length=0.05 radius=0.005
Joints:
- added joint M10FemurLinkage1.1: type revolute, parent M10ScrewFemur1.3, child M10LinkageFemur1.1_1, origin xyz=0 0 0 rpy=1.57 0 0 , axis 0 1 0, limit lower=1.352 upper=2.8715 effort=5000 velocity=1.0
- added joint M10KneeLinkage1.1: type revolute, parent M10Knee1.1, child M10LinkageFemur1.1_2, origin xyz=0 0 0.025 rpy=1.57 0 0 , axis 0 1 0, limit lower=1.352 upper=2.8715 effort=5000 velocity=1.0, mimic joint=M10FemurLinkage1.1 multiplier=-1 offset=0
- added joint SlideBlockM10_1.1: type fixed, parent SlideBlock1.1, child M10ScrewFemur1.1, origin xyz=0 -.05 0 rpy=1.57 0 0
- added joint SlideBlockM10_1.2: type fixed, parent SlideBlock1.1, child M10ScrewFemur1.2, origin xyz=0 .05 0 rpy=1.57 0 0
- added joint SlideBlockM10_1.3: type fixed, parent SlideBlock1.2, child M10ScrewFemur1.3, origin xyz=0 -.05 0 rpy=1.57 0 0
- added joint SlideBlockM10_1.4: type fixed, parent SlideBlock1.2, child M10ScrewFemur1.4, origin xyz=0 .05 0 rpy=1.57 0 0
